File: unibody_split.kicad_pcb (KiCad board)
At the start: 2 copper layers, 91 parts, among them U1 nice_nano

Commit message: Adds kbd library, wires everything up
Parts:
- removed SW_PWR1: SW_SPST, Button_Switch_THT:SW_Tactile_SPST_Angled_PTS645Vx31-2LFS
- added OL1: OLED, kbd:OLED_v2, F.Cu at (199.2, 146.8)
- D1, D10, D11, D12, D13, D14, D15, D16, D17, D18, D19, D2, D20, D21, D22, D23, D24, D25, D26, D27, D28, D29, D3, D30, D31, D32, D33, D34, D35, D36, D37, D38, D39, D4, D40, D41, D42, D43, D44, D5, D6, D7, D8, D9: moved to B.Cu
- moved D39 591.1 mm to (338.9, 151.6), turned to 90 degrees
- moved D43 586.5 mm to (358.0, 151.6), turned to 90 degrees
- moved D42 557.6 mm to (353.2, 132.6), turned to 90 degrees
- moved D41 555.0 mm to (350.8, 113.5), turned to 90 degrees
- moved D35 551.3 mm to (319.9, 151.6), turned to 90 degrees
- moved D44 546.4 mm to (350.8, 170.7), turned to 90 degrees
- moved D37 532.6 mm to (324.6, 113.5), turned to 90 degrees
- moved D38 522.5 mm to (329.4, 132.6), turned to 90 degrees
- moved D34 516.9 mm to (310.4, 132.6), turned to 90 degrees
- moved D40 516.0 mm to (319.9, 170.7), turned to 90 degrees
- moved D36 504.4 mm to (293.7, 170.7), turned to 90 degrees
- moved D33 503.6 mm to (305.6, 113.5), turned to 90 degrees
- moved D31 495.7 mm to (291.3, 132.6), turned to 90 degrees
- moved D30 481.5 mm to (286.5, 113.5), turned to 90 degrees
- moved D29 467.7 mm to (262.7, 170.7), turned to 90 degrees
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Connections:
- MX29 pad 1: COL7 -> COL6
- MX36 pad 1: unconnected-(MX36-Pad1) -> COL8
- MX40 pad 1: unconnected-(MX40-Pad1) -> COL9
- MX44 pad 1: unconnected-(MX44-Pad1) -> COL11
- U1 pad 10: ROW3 -> ROW1
- U1 pad 11: COL5 -> ROW2
- U1 pad 12: COL4 -> ROW3
- U1 pad 13: COL6 -> COL4
- U1 pad 14: COL7 -> COL5
- U1 pad 15: COL8 -> COL6
- U1 pad 16: PWR -> COL7
- U1 pad 17: COL9 -> COL8
- U1 pad 18: COL10 -> COL9
- U1 pad 19: COL11 -> COL10
- U1 pad 20: unconnected-(U1-Pad20) -> COL11
- U1 pad 5: COL2 -> SDA
- U1 pad 6: COL3 -> SCL
- U1 pad 7: ROW0 -> COL2
- U1 pad 8: ROW1 -> COL3
- U1 pad 9: ROW2 -> ROW0
Routing:
- net ROW3: track 0.00 -> 332.0 mm, vias 0 -> 14
- net ROW2: track 0.00 -> 317.4 mm, vias 0 -> 24
- net ROW0: track 0.00 -> 298.7 mm, vias 0 -> 22
- net ROW1: track 0.00 -> 294.9 mm, vias 0 -> 22
- net COL0: track 0.00 -> 204.9 mm, vias 0 -> 1
- net COL1: track 0.00 -> 202.2 mm, vias 0 -> 3
- net COL11: track 0.00 -> 186.4 mm, vias 0 -> 1
- net COL2: track 0.00 -> 160.2 mm, vias 0 -> 1
- net COL9: track 0.00 -> 146.9 mm, vias 0 -> 1
- net COL10: track 0.00 -> 146.3 mm, vias 0 -> 1
- net COL8: track 0.00 -> 132.2 mm, vias 0 -> 1
- net COL4: track 0.00 -> 129.0 mm, vias 0 -> 2
- net COL3: track 0.00 -> 121.4 mm, vias 0 -> 1
- net COL5: track 0.00 -> 97.2 mm, vias 0 -> 2
- net COL7: track 0.00 -> 91.0 mm, vias 0 -> 1
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Other:
- board outline added: 300 x 76.2 mm

Commit message: Adds ground plane, fixes edge cuts
Routing:
- added copper zone on B.Cu, net GND
- added copper zone on F.Cu, net GND
Other:
- board size 300 x 76.2 mm -> 302.4 x 81.7 mm
Changed lines of the file:
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@@
     )
   )
-  (gr_arc (start 60.325 101.6) (mid 61.022452 99.916202) (end 62.70625 99.21875) (layer "Edge.Cuts") (width 0.1))
-  (gr_line (start 62.70625 99.21875) (end 356.39375 99.21875) (layer "Edge.Cuts") (width 0.1))
-  (gr_line (start 357.1875 175.41875) (end 63.5 175.41875) (layer "Edge.Cuts") (width 0.1))
-  (gr_line (start 60.325 172.24375) (end 60.325 101.6) (layer "Edge.Cuts") (width 0.1))
-  (gr_arc (start 356.39375 99.21875) (mid 359.20008 100.38117) (end 360.3625 103.1875) (layer "Edge.Cuts") (width 0.1))
-  (gr_arc (start 63.5 175.41875) (mid 61.254936 174.488814) (end 60.325 172.24375) (layer "Edge.Cuts") (width 0.1))
-  (gr_line (start 360.3625 103.1875) (end 360.3625 172.24375) (layer "Edge.Cuts") (width 0.1))
-  (gr_arc (start 360.3625 172.24375) (mid 359.432564 174.488814) (end 357.1875 175.41875) (layer "Edge.Cuts") (width 0.1))
+  (gr_arc (start 59.162562 101.231298) (mid 60.325 98.425) (end 63.131312 97.262548) (layer "Edge.Cuts") (width 0.1))
+  (gr_line (start 59.162548 174.993688) (end 59.162562 101.231298) (layer "Edge.Cuts") (width 0.1))
+  (gr_line (start 361.524952 101.231312) (end 361.524938 174.993702) (layer "Edge.Cuts") (width 0.1))
+  (gr_arc (start 361.524938 174.993702) (mid 360.3625 177.8) (end 357.556188 178.962452) (layer "Edge.Cuts") (width 0.1))
+  (gr_line (start 357.556188 178.962452) (end 63.131298 178.962438) (layer "Edge.Cuts") (width 0.1))
+  (gr_arc (start 357.556202 97.262562) (mid 360.3625 98.425) (end 361.524952 101.231312) (layer "Edge.Cuts") (width 0.1))
+  (gr_arc (start 63.131298 178.962438) (mid 60.325 177.8) (end 59.162548 174.993688) (layer "Edge.Cuts") (width 0.1))
+  (gr_line (start 63.131312 97.262548) (end 357.556202 97.262562) (layer "Edge.Cuts") (width 0.1))
   (segment (start 238.194189 126.137061) (end 200.749561 126.137061) (width 0.25) (layer "F.Cu") (net 1))
   (segment (start 178.59375 123.03125) (end 180.49875 124.93625) (width 0.25) (layer "F.Cu") (net 1))
@@
   (segment (start 199.54875 117.31625) (end 196.85 120.015) (width 0.25) (layer "B.Cu") (net 70))
   (segment (start 196.85 143.1925) (end 199.23125 145.57375) (width 0.25) (layer "B.Cu") (net 70))
+  (zone (net 61) (net_name "GND") (layer "F.Cu") (hatch edge 0.508)
+    (connect_pads (clearance 0.508))
+    (min_thickness 0.254) (filled_areas_thickness no)
+    (fill yes (thermal_gap 0.508) (thermal_bridge_width 0.508))
+    (polygon
+      (pts
+        (xy 192.88125 111.91875)
+        (xy 182.5625 111.91875)
+        (xy 182.5625 103.1875)
+        (xy 192.88125 103.1875)
+      )
+    )
+  )
+  (zone (net 61) (net_name "GND") (layer "F.Cu") (hatch edge 0.508)
+    (connect_pads (clearance 0.508))
+    (min_thickness 0.254) (filled_areas_thickness no)
+    (fill yes (thermal_gap 0.508) (thermal_bridge_width 0.508))
+    (polygon
+      (pts
+        (xy 197.64375 111.91875)
+        (xy 192.88125 111.91875)
+        (xy 192.88125 108.74375)
+        (xy 197.64375 108.74375)
+      )
+    )
+  )
+  (zone (net 61) (net_name "GND") (layer "F.Cu") (hatch edge 0.508)
+    (connect_pads (clearance 0.508))
+    (min_thickness 0.254) (filled_areas_thickness no)
+    (fill yes (thermal_gap 0.508) (thermal_bridge_width 0.508))
+    (polygon
+      (pts
+        (xy 236.5375 153.19375)
+        (xy 197.64375 153.19375)
+        (xy 197.64375 140.49375)
+        (xy 236.5375 140.49375)
+      )
+    )
+  )
+  (zone (net 61) (net_name "GND") (layer "F.Cu") (hatch edge 0.508)
+    (connect_pads (clearance 0.508))
+    (min_thickness 0.254) (filled_areas_thickness no)
+    (fill yes (thermal_gap 0.508) (thermal_bridge_width 0.508))
+    (polygon
+      (pts
+        (xy 216.69375 134.9375)
+        (xy 197.64375 134.9375)
+        (xy 197.64375 100.0125)
+        (xy 216.69375 100.0125)
+      )
+    )
+  )
+  (zone (net 61) (net_name "GND") (layer "B.Cu") (hatch edge 0.508)
+    (connect_pads (clearance 0.508))
+    (min_thickness 0.254) (filled_areas_thickness no)
+    (fill yes (thermal_gap 0.508) (thermal_bridge_width 0.508))
+    (polygon
+      (pts
+        (xy 210.34375 146.84375)
+        (xy 209.55 146.84375)
+        (xy 209.55 153.19375)
+        (xy 197.64375 153.19375)
+        (xy 197.64375 146.84375)
+        (xy 201.6125 146.84375)
+        (xy 201.6125 113.50625)
+        (xy 198.4375 113.50625)
+        (xy 198.4375 108.74375)
+        (xy 210.34375 108.74375)
+      )
+    )
+  )
 )

Commit message: Adds smaller reset switch, JST for battery
Parts:
- removed SW_RESET1: SW_Push, random-keyboard-parts:SKQG-1155865
- added J1: Conn_01x02, Connector_JST:JST_PH_S2B-PH-SM4-TB_1x02-1MP_P2.00mm_Horizontal, B.Cu at (223.8, 105.6)
- added S1: EVP-AWBD2A, switches:SW_EVP-AWBD2A, F.Cu at (190.2, 108.4)
- added [MOUNT]: MountingHole_3.2mm_M3, MountingHole:MountingHole_3.2mm_M3, F.Cu at (330.2, 107.2)
- added [MOUNT]: MountingHole_3.2mm_M3, MountingHole:MountingHole_3.2mm_M3, F.Cu at (229.4, 170.7)
- added [MOUNT]: MountingHole_3.2mm_M3, MountingHole:MountingHole_3.2mm_M3, F.Cu at (187.3, 170.7)
- added [MOUNT]: MountingHole_3.2mm_M3, MountingHole:MountingHole_3.2mm_M3, F.Cu at (180.2, 108.7)
- added [MOUNT]: MountingHole_3.2mm_M3, MountingHole:MountingHole_3.2mm_M3, F.Cu at (82.9, 120.3)
- added [MOUNT]: MountingHole_3.2mm_M3, MountingHole:MountingHole_3.2mm_M3, F.Cu at (84.8, 163.7)
- added [MOUNT]: MountingHole_3.2mm_M3, MountingHole:MountingHole_3.2mm_M3, F.Cu at (327.8, 163.5)
Routing:
- net BATT_IN: track 0.00 -> 14.1 mm
- net BATT_GND: track 0.00 -> 9.89 mm
- net GND: track 0.00 -> 8.31 mm
- net RESET: track 32.1 -> 27.1 mm
- net COL1: track 202.2 -> 202.5 mm, vias 3 -> 2
Other:
- board text added: "Spank Me!"

Commit message: Update JST header to XH
Parts:
- J1: footprint Connector_JST:JST_PH_S2B-PH-SM4-TB_1x02-1MP_P2.00mm_Horizontal -> Connector_JST:JST_XH_S2B-XH-A_1x02_P2.50mm_Horizontal
- moved J1 21.4 mm to (223.8, 127.0)
Routing:
- net COL6: track 88.1 -> 0.00 mm, vias 1 -> 0
- net ROW0: track 298.7 -> 386.8 mm, vias 22 -> 23
- net BATT_GND: track 9.89 -> 25.4 mm
- net BATT_IN: track 14.1 -> 29.5 mm
