File: unibody_split.kicad_pcb (KiCad board)
At the start: 2 copper layers, 305.5 x 82.5 mm, 92 parts, among them J1 Conn_01x02, U1 nice_nano

Commit message: Move nice nano to new board edge, zone fills
Parts:
- S1: footprint switches:SW_EVP-AWBD2A -> random-keyboard-parts:SKQG-1155865
- moved U1 3.89 mm to (207.2, 114.7)
Routing:
- net ROW1: track 282.1 -> 292.6 mm, vias 22 -> 24
- net ROW3: track 329.2 -> 339.5 mm, vias 8 -> 9
- net ROW2: track 307.4 -> 315.5 mm
- net ROW0: track 290.2 -> 284.5 mm
- net VCC: track 48.6 -> 52.4 mm
- net SDA: track 29.4 -> 33.3 mm
- net SCL: track 30.4 -> 34.2 mm
- net COL5: track 97.2 -> 101.1 mm
- net COL4: track 129.0 -> 132.9 mm
- net COL10: track 145.4 -> 142.5 mm
- net GND: track 8.31 -> 10.7 mm
- net COL1: track 202.5 -> 204.9 mm
- net BATT_GND: track 24.9 -> 26.7 mm
- net BATT_IN: track 28.5 -> 30.1 mm
- net COL7: track 91.0 -> 89.4 mm
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