File: _autosave-unibody_split.kicad_pcb (KiCad board)
At the start: 2 copper layers, 302.4 x 79.7 mm, 99 parts, among them J1 Conn_01x02, U1 nice_nano

Commit message: Use sma diodes
Parts:
- removed [MOUNT] (x7): MountingHole_3.2mm_M3, MountingHole:MountingHole_3.2mm_M3
- D1, D10, D11, D12, D13, D14, D15, D16, D17, D18, D19, D2, D20, D21, D22, D23, D24, D25, D26, D27, D28, D29, D3, D30, D31, D32, D33, D34, D35, D36, D37, D38, D39, D4, D40, D41, D42, D43, D44, D5, D6, D7, D8, D9: footprint digikey-footprints:DO-214AC -> Diode_SMD:D_SMA_Handsoldering
- moved D19 11.2 mm to (175.3, 166.0)
- moved D12 2.38 mm to (134.1, 170.7)
- moved D18 2.38 mm to (169.9, 151.6)
- moved D25 2.38 mm to (265.1, 151.6)
- moved D26 2.38 mm to (269.9, 113.5)
- moved D28 2.38 mm to (284.2, 151.6)
- moved D29 2.38 mm to (265.1, 170.7)
- moved D30 2.38 mm to (288.9, 113.5)
- moved D31 2.38 mm to (293.7, 132.6)
- moved D33 2.38 mm to (308.0, 113.5)
- moved D34 2.38 mm to (312.7, 132.6)
- moved D36 2.38 mm to (296.1, 170.7)
- moved D38 2.38 mm to (331.8, 132.6)
- moved D39 2.38 mm to (341.3, 151.6)
- moved D41 2.38 mm to (353.2, 113.5)
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Routing:
- net ROW2: track 649.4 -> 311.0 mm, vias 38 -> 20
- net ROW3: track 0.00 -> 328.6 mm, vias 0 -> 8
- net ROW0: track 0.00 -> 290.2 mm, vias 0 -> 24
- net COL6: track 90.2 -> 142.6 mm
- net BATT_IN: track 29.5 -> 0.00 mm
- net BATT_GND: track 25.1 -> 0.00 mm
- net ROW1: track 294.9 -> 285.7 mm
- net Net-(D37-Pad2): track 8.73 -> 0.00 mm
- net Net-(D33-Pad2): track 8.73 -> 0.00 mm
- net Net-(D23-Pad2): track 8.73 -> 0.00 mm
- net Net-(D30-Pad2): track 8.73 -> 0.00 mm
- net Net-(D26-Pad2): track 8.73 -> 0.00 mm
- net Net-(D19-Pad2): track 8.73 -> 12.6 mm
- net Net-(D10-Pad2): track 8.73 -> 10.4 mm
- net Net-(D17-Pad2): track 8.73 -> 10.4 mm
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